File: dc-to-dc-maker/Converter DCAC/Converter DCAC.kicad_sch (KiCad schematic)
At the start: 18 parts, among them Q1 IRF640NPBF, Q2 IRF640NPBF, Q3 IRF640NPBF, Q4 IRF640NPBF, U1 IR2110PBF

Commit message: Add files via upload
Parts:
- added C3: 100n, symbol Device:C
Connections:
- net GND: now also C3.2
- net at U1.11 (SD), U1.3 (VCC), U1.9 (VDD)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: now also C3.1
Changed lines of the file:
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@@
 	)
 	(junction
-		(at 129.54 58.42)
+		(at 130.81 58.42)
 		(diameter 0)
 		(color 0 0 0 0)
@@
 	)
 	(junction
+		(at 118.11 64.77)
+		(diameter 0)
+		(color 0 0 0 0)
+	)
+	(junction
 		(at 135.89 107.95)
 		(diameter 0)
@@
 	)
 	(junction
+		(at 134.62 64.77)
+		(diameter 0)
+		(color 0 0 0 0)
+	)
+	(junction
 		(at 92.71 64.77)
 		(diameter 0)
@@
 	(wire
 		(pts
+			(xy 107.95 60.96) (xy 118.11 60.96)
+		)
+		(stroke
+			(width 0)
+			(type default)
+		)
+	)
+	(wire
+		(pts
 			(xy 78.74 54.61) (xy 105.41 54.61)
 		)
@@
 	(wire
 		(pts
-			(xy 125.73 64.77) (xy 125.73 63.5)
-		)
-		(stroke
-			(width 0)
-			(type default)
-		)
-	)
-	(wire
-		(pts
 			(xy 144.78 135.89) (xy 144.78 140.97)
 		)
@@
 	(wire
 		(pts
+			(xy 134.62 64.77) (xy 137.16 64.77)
+		)
+		(stroke
+			(width 0)
+			(type default)
+		)
+	)
+	(wire
+		(pts
 			(xy 66.04 181.61) (xy 69.85 181.61)
 		)
@@
 	(wire
 		(pts
-			(xy 129.54 58.42) (xy 130.81 58.42)
-		)
-		(stroke
-			(width 0)
-			(type default)
-		)
-	)
-	(wire
-		(pts
 			(xy 135.89 107.95) (xy 149.86 107.95)
 		)
@@
 	(wire
 		(pts
+			(xy 130.81 64.77) (xy 134.62 64.77)
+		)
+		(stroke
+			(width 0)
+			(type default)
+		)
+	)
+	(wire
+		(pts
 			(xy 129.54 125.73) (xy 124.46 125.73)
 		)
@@
 	(wire
 		(pts
+			(xy 134.62 53.34) (xy 134.62 64.77)
+		)
+		(stroke
+			(width 0)
+			(type default)
+		)
+	)
+	(wire
+		(pts
 			(xy 113.03 44.45) (xy 116.84 44.45)
 		)
@@
 	(wire
 		(pts
+			(xy 107.95 53.34) (xy 134.62 53.34)
+		)
+		(stroke
+			(width 0)
+			(type default)
+		)
+	)
+	(wire
+		(pts
 			(xy 119.38 107.95) (xy 119.38 109.22)
 		)
@@
 	(wire
 		(pts
-			(xy 137.16 64.77) (xy 130.81 64.77)
-		)
-		(stroke
-			(width 0)
-			(type default)
-		)
-	)
-	(wire
-		(pts
 			(xy 130.81 107.95) (xy 135.89 107.95)
 		)
@@
 	(wire
 		(pts
-			(xy 129.54 38.1) (xy 129.54 58.42)
+			(xy 130.81 38.1) (xy 130.81 58.42)
+		)
+		(stroke
+			(width 0)
+			(type default)
+		)
+	)
+	(wire
+		(pts
+			(xy 125.73 63.5) (xy 125.73 64.77)
 		)
 		(stroke
@@
 	(wire
 		(pts
-			(xy 66.04 38.1) (xy 129.54 38.1)
+			(xy 66.04 38.1) (xy 130.81 38.1)
 		)
 		(stroke
@@
 	(wire
 		(pts
+			(xy 118.11 60.96) (xy 118.11 64.77)
+		)
+		(stroke
+			(width 0)
+			(type default)
+		)
+	)
+	(wire
+		(pts
 			(xy 135.89 116.84) (xy 135.89 128.27)
 		)
@@
 	(wire
 		(pts
-			(xy 120.65 58.42) (xy 129.54 58.42)
+			(xy 120.65 58.42) (xy 130.81 58.42)
 		)
 		(stroke
@@
 					(unit 1)
 				)
+			)
+		)
+	)
+	(symbol
+		(lib_id "Device:C")
+		(at 107.95 57.15 0)
+		(unit 1)
+		(exclude_from_sim no)
+		(in_bom yes)
+		(on_board yes)
+		(dnp no)
+		(fields_autoplaced yes)
+		(property "Reference" "C3"
+			(at 111.76 55.8799 0)
+			(effects
+				(font
+					(size 1.27 1.27)
+				)
+				(justify left)
+			)
+		)
+		(property "Value" "100n"
+			(at 111.76 58.4199 0)
+			(effects
+				(font
+					(size 1.27 1.27)
+				)
+				(justify left)
+			)
+		)
+		(property "Footprint" ""
+			(at 108.9152 60.96 0)
+			(effects
+				(font
+					(size 1.27 1.27)
+				)
+				(hide yes)
+			)
+		)
+		(property "Datasheet" "~"
+			(at 107.95 57.15 0)
+			(effects
+				(font
+					(size 1.27 1.27)
+				)
+				(hide yes)
+			)
+		)
+		(property "Description" "Unpolarized capacitor"
+			(at 107.95 57.15 0)
+			(effects
+				(font
+					(size 1.27 1.27)
+				)
+				(hide yes)
+			)
+		)
+		(pin "2"
+		)
+		(pin "1"
+		)
+		(instances
+			(project "Converter DCAC"
+				(path "/1fde7b99-6848-43ce-ad86-15bc0c96cf11"
+					(reference "C3")
+					(unit 1)
+				)

Commit message: Add files via upload
Parts:
- added C4: 100n, symbol Device:C
- added D2: D, symbol Device:D
- added J1: 1715734, 1715734:PHOENIX_1715734, symbol 1715734:1715734
- added U2: LA55-P, Sensor_Current:LEM_LA25-P, symbol Sensor_Current:LA55-P
Connections:
- net GND: now also C4.2, D2.2 (A)
- net at C1.2, U1.6 (VB): now also C4.1, D2.1 (K)
- new net: J1.1, U2.3 (+)
- new net: J1.2, U2.2 (-)
- new net: J1.3, U2.1 (M)
