File: dc-to-dc-maker/dc-to-dc-buck-converter/dc-to-dc-buck-converter.kicad_pcb (KiCad board)
At the start: 2 copper layers, 1 part, among them U1 IRF640NPBF

Commit message: pcb structure + images
Parts:
- removed U1: IRF640NPBF, IRF640NPBF:TO254P483X1016X1994-3P
- added REF**: MountingHole_6mm_Pad_Via, MountingHole:MountingHole_6mm_Pad_Via, F.Cu at (191.7, 65.3)
- added REF**: MountingHole_6mm_Pad_Via, MountingHole:MountingHole_6mm_Pad_Via, F.Cu at (104.7, 65.3)
- added REF**: MountingHole_6mm_Pad_Via, MountingHole:MountingHole_6mm_Pad_Via, F.Cu at (191.7, 132.3)
- added REF**: MountingHole_6mm_Pad_Via, MountingHole:MountingHole_6mm_Pad_Via, F.Cu at (104.7, 132.3)
Other:
- board outline added: 100 x 80 mm

Commit message: update to pcb placement
Parts:
- added C1: 0.1uF, C322C104K5R5TA(decoup capacitor):C322, F.Cu at (113.8, 66.7)
- added C10: 220uF, EEUFC1J221S(capacitor):CAPPRD500W65D1250H2200, F.Cu at (142.8, 105.7)
- added C2: 0.1uF, C322C104K5R5TA(decoup capacitor):C322, F.Cu at (113.8, 71.2)
- added C3: 0.1uF, C322C104K5R5TA(decoup capacitor):C322, F.Cu at (133.3, 89.2)
- added C4: 0.1uF, C322C104K5R5TA(decoup capacitor):C322, F.Cu at (168.8, 66.2)
- added C5: 0.1uF, C322C104K5R5TA(decoup capacitor):C322, F.Cu at (130.8, 113.2)
- added C6: 0.1uF, C322C104K5R5TA(decoup capacitor):C322, F.Cu at (133.3, 93.2)
- added C7: 0.1uF, C322C104K5R5TA(decoup capacitor):C322, F.Cu at (187.3, 66.7)
- added C8: 0.1uF, C322C104K5R5TA(decoup capacitor):C322, F.Cu at (187.3, 70.7)
- added C9: 0.1uF, C322C104K5R5TA(decoup capacitor):C322, F.Cu at (186.3, 94.7)
- added D1: MBR10100+, MBR10100+(diode):TO490P480X1000X2110-2P, F.Cu at (161.2, 102.2)
- added IC1: LA_55-P, LA_55-P(current detector):LA55-P, F.Cu at (136.3, 57.2)
- added IC2: LA_55-P, LA_55-P(current detector):LA55-P, F.Cu at (162.7, 122.2)
- added IC3: EL7104CNZ, EL7104CNZ(voltage regulator):DIP762W51P254L952H533Q8N, F.Cu at (146.1, 90.7)
- added J1: Conn_01x06_Pin, Connector_Harwin:Harwin_M20-89006xx_1x06_P2.54mm_Horizontal, F.Cu at (108.3, 89.9)
- added J2: Jgen, 1715721(screw connector):1715721, F.Cu at (118.1, 57.0)
- added J3: Jaux 9V, 1715721(screw connector):1715721, F.Cu at (182.5, 56.4)
- added J4: Jind, 1715721(screw connector):1715721, F.Cu at (182.3, 122.7)
- added J5: Jout +50V, 1715721(screw connector):1715721, F.Cu at (193.1, 86.9)
- added LED1: TLUR5400, TLUR5400(led):TLUR5400, F.Cu at (190.1, 108.7)
- added R1: 20K, MF25_20K(resistor):RESAD1680W59L680D250, F.Cu at (120.8, 89.7)
- added R2: 1K, MF25_1K(resistor):RESAD1680W59L680D250, F.Cu at (120.8, 109.6)
- added R3: 100, MF25_100R(resistor):RESAD1680W59L680D250, F.Cu at (126.3, 89.6)
- added R4: 100, MF25_100R(resistor):RESAD1680W59L680D250, F.Cu at (126.3, 109.6)
- added R5: 10, MF25_10R(resistor):RESAD1680W59L680D250, F.Cu at (155.2, 89.2)
- added R6: 10, MF25_10R(resistor):RESAD1680W59L680D250, F.Cu at (161.9, 112.2)
- added R7: 20K, MF25_20K(resistor):RESAD1680W59L680D250, F.Cu at (178.8, 89.6)
- added R8: 1K, MF25_1K(resistor):RESAD1680W59L680D250, F.Cu at (178.8, 108.7)
- added U1: IRF640NPBF, IRF640NPBF(mosfet):TO254P483X1016X1994-3P, F.Cu at (161.1, 96.2)
- 1MH_6mm, 2MH_6mm, 3MH_6mm, 4MH_6mm: renamed from REF**; value MountingHole_6mm_Pad_Via -> MH_6mm
- moved 1MH_6mm 9.00 mm to (106.5, 56.5)
- moved 3MH_6mm 9.00 mm to (193.5, 56.5)
- moved 2MH_6mm 9.00 mm to (106.5, 123.5)
- moved 4MH_6mm 9.00 mm to (193.5, 123.5)
Routing:
- added copper zone on B.Cu, net GND
Other:
- board text added: "Group 10 Electrical Warriors"
- board text added: "Jaux9V"
- board text added: "Jgen"
- board text added: "Jind"
- board text added: "Jout50V"

Commit message: pcb final
Parts:
- removed J1: Conn_01x06_Pin, Connector_Harwin:Harwin_M20-89006xx_1x06_P2.54mm_Horizontal
- added Jmc1: 1715734, 1715734(screw connector):1715734, F.Cu at (173.0, 78.1)
- added Jmc2: 1715734, 1715734(screw connector):1715734, F.Cu at (142.6, 57.0)
- Jaux: renamed from J3; value Jaux 9V -> Jaux
- moved Jind 77.3 mm to (106.7, 106.8), turned to -90 degrees
- moved R4 71.0 mm to (182.0, 65.6), turned to -90 degrees
- moved J5out 68.9 mm to (134.5, 123.0), turned to 0 degrees
- moved C7 63.3 mm to (127.5, 87.5)
- moved R2 56.8 mm to (115.5, 53.0), turned to -90 degrees
- moved C8 54.4 mm to (135.5, 87.5), turned to 180 degrees
- moved C6 53.9 mm to (176.5, 61.0), turned to 180 degrees
- moved U1 45.9 mm to (119.9, 116.5)
- moved C9 45.9 mm to (146.5, 117.5), turned to 90 degrees
- moved D1 42.3 mm to (125.0, 124.0), turned to 180 degrees
- moved C5 39.0 mm to (168.5, 123.0), turned to 90 degrees
- moved Jgen 37.6 mm to (106.7, 92.8), turned to -90 degrees
- moved R1 27.6 mm to (103.0, 68.6), turned to -90 degrees
- moved IC1 27.6 mm to (155.5, 77.0), turned to 0 degrees
- moved R6 25.3 mm to (165.5, 87.1), turned to -90 degrees
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- renumbered J5 to J5out, J2 to Jgen, J4 to Jind
Connections:
- C5 pad 1: Net-(IC2-POS) -> Net-(IC1-POS)
- IC2 pad 3: Net-(IC2-POS) -> Net-(IC1-POS)
Routing:
- net Net-(C3-Pad1): track 0.00 -> 119.5 mm
- net Net-(IC3-IN): track 0.00 -> 88.5 mm
- net Net-(IC1-M): track 0.00 -> 58.2 mm, vias 0 -> 4
- net Net-(C6-Pad1): track 0.00 -> 50.8 mm
- net Net-(Jmc2-Pad3): track 0.00 -> 36.5 mm
- net Net-(IC3-N_OUT): track 0.00 -> 22.6 mm
- net Net-(IC2-M): track 0.00 -> 11.0 mm
- net Net-(U1-GATE): track 0.00 -> 10.1 mm
- net Net-(LED1-A): track 0.00 -> 6.64 mm
- added copper zone on F.Cu, net Net-(C1-Pad2)
- added copper zone on F.Cu, net Net-(C10-+)
- added copper zone on F.Cu, net Net-(D1-A)
- added copper zone on B.Cu, net Net-(IC1-POS)
- added copper zone on F.Cu, net Net-(IC1-POS)
- added copper zone on F.Cu, net Net-(Jmc1-Pad1)
Other:
- board text added: "Group 10 Wireless Warriors"
- board text removed: "Group 10 Electrical Warriors"
- board text removed: "Jaux9V"
- board text removed: "Jgen"
- board text removed: "Jind"
- board text removed: "Jout50V"
