File: dc-to-dc-maker/dc-to-dc-buck-converter/dc-to-dc-buck-converter.kicad_sch (KiCad schematic)
At the start: 10 parts, among them IC1 EL7104CNZ, J1 1715721, J2 1715721, J3 1-826629-6, U1 IRF640NPBF

Commit message: pcb structure + images
Connections:
- net at R1.2: now also U1.1 (GATE)
Other:
- note added: "- check mosfet driver schematic - ensure max 5V between pins and mosfet driver (voltage divider) - pinout structure for impedance - mosfet connections confirmation - check circuit and finish"
- moved on the sheet: C1, U1

Commit message: updates
Connections:
- net at D1.1 (K): now also U1.2 (SOURCE)
Other:
- note added: "low pass rc filter"

Commit message: update
Parts:
- removed C2: EEUFC1J221S, EEUFC1J221S(capacitor):CAPPRD500W65D1250H2200, symbol EEUFC1J221S(capacitor):EEUFC1J221S
- removed D1: MBR10100+, MBR10100+(diode):TO490P480X1000X2110-2P, symbol MBR10100+(diode):MBR10100+
- removed IC1: EL7104CNZ, EL7104CNZ(voltage regulator):DIP762W51P254L952H533Q8N, symbol EL7104CNZ(voltage regulator):EL7104CNZ
- removed J2: 1715721, 1715721(screw connector):1715721, symbol 1715721(screw connector):1715721
- removed J3: 1-826629-6, 1-826629-6(pins):HDRV16W63P0X254_1X16_4064X250X950P, symbol 1-826629-6(pins):1-826629-6
- removed R1: MF25_10R, RESAD1680W59L680D250, symbol MF25_10R(resistor):MF25_10R
- removed U1: IRF640NPBF, IRF640NPBF(mosfet):TO254P483X1016X1994-3P, symbol IRF640NPBF(mosfet):IRF640NPBF
- added C10, C2, C4, C5, C6, C7, C8: 0.1uF, C322C104K5R5TA(decoup capacitor):C322, symbol C322C104K5R5TA(decoup capacitor):C322C104K5R5TA
- added C9: 220uF, EEUFC1J221S(capacitor):CAPPRD500W65D1250H2200, symbol EEUFC1J221S(capacitor):EEUFC1J221S
- added D1: LED, symbol Device:LED
- added D2: MBR10100+, MBR10100+(diode):TO490P480X1000X2110-2P, symbol MBR10100+(diode):MBR10100+
- added IC1, IC3: LA_55-P, LA_55-P(current detector):LA55-P, symbol LA_55-P(current-sensor):LA_55-P
- added IC2: EL7104CNZ, EL7104CNZ(voltage regulator):DIP762W51P254L952H533Q8N, symbol EL7104CNZ(voltage regulator):EL7104CNZ
- added J3: Jgen, 1715721(screw connector):1715721, symbol 1715721(screw connector):1715721
- added J4: STM_PinS, Connector_Hirose:Hirose_DF63M-1P-3.96DSA_1x01_P3.96mm_Vertical, symbol Connector:Conn_01x06_Pin
- added J5: Jaux 9V, 1715721(screw connector):1715721, symbol 1715721(screw connector):1715721
- added J6: Jind, 1715721(screw connector):1715721, symbol 1715721(screw connector):1715721
- added R1, R2: 20K, MF25_20K(resistor):RESAD1680W59L680D250, symbol MF25_20K(resistor):MF25_20K
- added R3, R6: 1K, MF25_1K(resistor):RESAD1680W59L680D250, symbol MF25_1K(resistor):MF25_1K
- added R4, R8: 100, RESAD1680W59L680D250, symbol MF25_100R(resistor):MF25_100R
- added R5, R7: 10, RESAD1680W59L680D250, symbol MF25_10R(resistor):MF25_10R
- added U2: IRF640NPBF, IRF640NPBF(mosfet):TO254P483X1016X1994-3P, symbol IRF640NPBF(mosfet):IRF640NPBF
- C1, C3: value C322C104K5R5TA -> 0.1uF
- J1: value 1715721 -> Jout +50V
Connections:
- net GND: now also C1.1, C10.2, C2.2, C4.1, C5.2, C6.1, C7.1, C8.2, C9.2 (-), D1.1 (K), IC1.2 (NEG), IC2.4 (GND_1), IC2.5 (GND_2), IC3.2 (NEG), J3.2, J4.1 (Pin_1), J5.2, R3.1, R6.1, U2.3 (DRAIN)
- net at C1.2: now also C4.2, J3.1, J6.1, R2.2
- net VDC: no longer names the net of C3.2, J1.1
- net VDC: now also C9.1 (+), D2.1 (K), R1.2
- new net: C5.1, C6.2, C7.2, IC2.1 (V+_1), IC2.8 (V+_2), IC3.3 (POS), J5.1
- new net: C10.1, IC1.3 (POS)
- new net: J4.4 (Pin_4), R2.1, R3.2
- new net: IC2.6 (N_OUT), IC2.7 (P_OUT), R5.1
- new net: R5.2, U2.2 (SOURCE)
- new net: J4.5 (Pin_5), R1.1, R6.2, R7.1
- new net: D2.2 (A), J6.2, U2.1 (GATE)
- new net: IC1.1 (M), R8.2
- new net: C8.1, J4.2 (Pin_2), R4.1
- new net: C2.1, J4.6 (Pin_6), R8.1
- new net: IC3.1 (M), R4.2
- new net: IC2.2 (IN), J4.3 (Pin_3)
- new net: D1.2 (A), R7.2
Other:
- note removed: "- check mosfet driver schematic - ensure max 5V between pins and mosfet driver (voltage divider) - pinout structure for impedance - mosfet connections confirmation - check circuit and finish"
- note removed: "low pass rc filter"
- title: DC to DC Buck Boost Converter -> DC to DC Boost Converter
- moved on the sheet: C1

Commit message: update to pcb placement
Parts:
- removed D1: LED, symbol Device:LED
- removed J4: STM_PinS, Connector_Hirose:Hirose_DF63M-1P-3.96DSA_1x01_P3.96mm_Vertical, symbol Connector:Conn_01x06_Pin
- added J1: Conn_01x06_Pin, Connector_Harwin:Harwin_M20-89006xx_1x06_P2.54mm_Horizontal, symbol Connector:Conn_01x06_Pin
- added LED1: TLUR5400, TLUR5400(led):TLUR5400, symbol TLUR5400(led):TLUR5400
- R3: renamed from R4; footprint RESAD1680W59L680D250 -> MF25_100R(resistor):RESAD1680W59L680D250
- R4: renamed from R8; footprint RESAD1680W59L680D250 -> MF25_100R(resistor):RESAD1680W59L680D250
- R5: footprint RESAD1680W59L680D250 -> MF25_10R(resistor):RESAD1680W59L680D250
- R6: renamed from R7; footprint RESAD1680W59L680D250 -> MF25_10R(resistor):RESAD1680W59L680D250
- renumbered C9 to C10, C4 to C2, C8 to C3, C5 to C4, C10 to C5, C2 to C6, C6 to C7, C7 to C8, C3 to C9, D2 to D1, IC3 to IC1, IC1 to IC2, IC2 to IC3, J3 to J2, J5 to J3, J6 to J4, J1 to J5, R2 to R1, R3 to R2, R1 to R7, R6 to R8, U2 to U1
Connections:
- net GND: now also U1.2 (SOURCE), J1.1 (Pin_1), LED1.2 (K); no longer U1.3 (DRAIN)
- net at R1.1, R2.2: now also J1.4 (Pin_4)
- net at R5.2: now also U1.1 (GATE); no longer U1.2 (SOURCE)
- net at R6.1, R7.1, R8.2: now also J1.5 (Pin_5)
- net at D1.2 (A), J4.2: now also U1.3 (DRAIN); no longer U1.1 (GATE)
- net at C3.1, R3.1: now also J1.2 (Pin_2)
- net at C6.1, R4.1: now also J1.6 (Pin_6)
- net at IC3.2 (IN): now also J1.3 (Pin_3)
- net at R6.2: now also LED1.1 (A)

Commit message: pcb final
Parts:
- removed J1: Conn_01x06_Pin, Connector_Harwin:Harwin_M20-89006xx_1x06_P2.54mm_Horizontal, symbol Connector:Conn_01x06_Pin
- added Jmc1, Jmc2: 1715734, 1715734(screw connector):1715734, symbol 1715734(screw connector):1715734
Connections:
- net GND: now also Jmc1.3
- net at C4.1, C7.2, C8.2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: now also C5.1, IC2.3 (POS)
- net at R1.1, R2.2: now also Jmc2.3
- net at R6.1, R7.1, R8.2: now also Jmc1.1
- net at C3.1, R3.1: now also Jmc2.2
- net at IC3.2 (IN): now also Jmc1.2
- net at C6.1, R4.1: now also Jmc2.1
