File: dc-to-dc-maker/dc-to-dc-boost-converter/dc-to-dc-buck-converter.kicad_pcb (KiCad board)
At the start: 2 copper layers, 100 x 80 mm, 34 parts, among them IC1 LA_55-P, IC2 LA_55-P, IC3 EL7104CNZ, J5out Jout +50V, U1 IRF640NPBF

Commit message: update
Parts:
- renumbered Jaux to Jaux9V, J5out to Jout50V
Changed lines of the file:
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@@
 	(paper "A4")
 	(title_block
-		(title "DC to DC Buck Boost Converter")
+		(title "DC to DC Boost Converter")
 		(date "2024-05-16")
 		(company "CBL Team 10")
@@
 		(descr "1715721")
 		(tags "Connector")
-		(property "Reference" "Jaux"
+		(property "Reference" "Jaux9V"
 			(at 2.83 -3.7 0)
 			(layer "F.SilkS")
@@
 		(tags "Resistor")
 		(property "Reference" "R3"
-			(at 0 0 90)
+			(at 8.4 0 180)
 			(layer "F.SilkS")
 			(effects
@@
 		(tags "Resistor")
 		(property "Reference" "R2"
-			(at 15.5 -2.75 180)
+			(at 8.4 0 180)
 			(layer "F.SilkS")
 			(effects
@@
 		(tags "Capacitor Polarised")
 		(property "Reference" "C10"
-			(at 0 0 90)
+			(at 2.5 0 180)
 			(layer "F.SilkS")
 			(effects
@@
 		(tags "Capacitor")
 		(property "Reference" "C2"
-			(at -0.3 -0.044 90)
+			(at -0.3 -0.044 180)
 			(layer "F.SilkS")
 			(effects
@@
 		(tags "Capacitor")
 		(property "Reference" "C1"
-			(at -0.3 0 90)
+			(at -0.3 0 180)
 			(layer "F.SilkS")
 			(effects
@@
 		(descr "1715721")
 		(tags "Connector")
-		(property "Reference" "J5out"
+		(property "Reference" "Jout50V"
 			(at 2.5 3 0)
 			(layer "F.SilkS")
@@
 		(tags "Integrated Circuit")
 		(property "Reference" "IC2"
-			(at -14.4 -0.2 90)
+			(at -14.4 -0.2 180)
 			(layer "F.SilkS")
 			(effects
@@
 		(tags "Capacitor")
 		(property "Reference" "C5"
-			(at -0.3 -0.044 -90)
+			(at -0.3 -0.044 0)
 			(layer "F.SilkS")
 			(effects
@@
 		(tags "Capacitor")
 		(property "Reference" "C9"
-			(at -0.3 -0.044 -90)
+			(at -0.3 -0.044 0)
 			(layer "F.SilkS")
 			(effects
@@
 			(pts
 				(xy 127 90.5) (xy 126 91) (xy 126 93) (xy 126.75 93.5) (xy 128.75 93.5) (xy 129.25 93) (xy 134.25 93)
-				(xy 134.5 93.5) (xy 136.25 93.5) (xy 136.75 93) (xy 136.75 86) (xy 144 83.25) (xy 156.25 79) (xy 157.75 77.75)
-				(xy 163 60.5) (xy 164.25 59.75) (xy 164.25 57) (xy 163.5 56.5) (xy 160.75 56.5) (xy 160.25 57) (xy 149.25 65.25)
-				(xy 144 70.5) (xy 133.25 79.25) (xy 127.25 81)
+				(xy 134.5 93.5) (xy 136.25 93.5) (xy 136.75 93) (xy 135.25 85.91) (xy 144 83) (xy 156.25 79) (xy 157.75 77.75)
+				(xy 163 60.5) (xy 164.25 59.75) (xy 164.25 57) (xy 163.5 56.5) (xy 160.5 56.25) (xy 159.75 57) (xy 149.75 65.75)
+				(xy 144.25 70.75) (xy 133.75 79.75) (xy 127.25 81)
 			)
 		)
@@
 		(polygon
 			(pts
-				(xy 175.5 77) (xy 175.5 87.5) (xy 173.5 88.5) (xy 160 88.5) (xy 158.5 87.5) (xy 158.5 85) (xy 160 84)
-				(xy 170.5 84) (xy 170.5 77) (xy 171.5 76) (xy 174.5 76)
+				(xy 175.5 77) (xy 175.5 87.5) (xy 173.5 88.5) (xy 160 88.5) (xy 158 87.5) (xy 158 85) (xy 158 84)
+				(xy 162.25 79.5) (xy 165.25 76) (xy 171.5 76) (xy 174.5 76)
 			)
 		)
@@
 		(polygon
 			(pts
-				(xy 104.25 108) (xy 105.25 108.75) (xy 108.25 108.75) (xy 109.25 108.25) (xy 116.25 112.25) (xy 123.25 105.75)
-				(xy 119.75 102.25) (xy 119.75 83.5) (xy 117.25 82.25) (xy 104 82.25) (xy 101.5 83.5) (xy 101.5 93.5)
-				(xy 109.75 96.5) (xy 104.25 105)
+				(xy 104.25 108) (xy 105.25 108.75) (xy 108.25 108.75) (xy 109 109.5) (xy 116.5 113) (xy 122 107.25)
+				(xy 119.25 102) (xy 118.91 83.55) (xy 117.25 82.25) (xy 104 82.25) (xy 101.5 83.5) (xy 101.5 95.25)
+				(xy 110.5 95.25) (xy 104.25 105)
 			)
 		)
@@
 		(polygon
 			(pts
-				(xy 105.25 110) (xy 104.75 111) (xy 104.75 115.5) (xy 109.5 116.75) (xy 117.5 125.25) (xy 120.5 126.25)
-				(xy 122.55 124.8) (xy 122.75 120.75) (xy 127 118) (xy 127 115.5) (xy 126 114.25) (xy 124.25 114.25)
-				(xy 123.5 115.25) (xy 123.5 118.25) (xy 116.5 118) (xy 116.5 113.5) (xy 108.75 110)
+				(xy 105.25 110) (xy 104.75 111) (xy 104.75 115.5) (xy 110 115.5) (xy 117.3 124.8) (xy 120 126.25)
+				(xy 122.55 124.8) (xy 122.5 120.5) (xy 127 118) (xy 127 115.25) (xy 126.5 114.25) (xy 124.25 114.25)
+				(xy 123.75 115.25) (xy 123.75 118) (xy 116.5 118) (xy 116.5 113.5) (xy 108.75 110)
 			)
 		)
@@
 				(xy 182 123) (xy 180.5 123.5) (xy 178 123.5) (xy 170.5 126.25) (xy 169.5 127) (xy 167.25 127) (xy 166 126.25)
 				(xy 157 111) (xy 152.75 103) (xy 136.75 93) (xy 136.25 93.5) (xy 134.5 93.5) (xy 134.25 93) (xy 129.25 93)
-				(xy 128.75 93.5) (xy 126.75 93.5) (xy 126 93) (xy 126 91) (xy 127 90.5) (xy 127.25 81) (xy 133.25 79.25)
-				(xy 144 70.5) (xy 160.75 56.5) (xy 163.5 56.5) (xy 164.25 57) (xy 164.25 59.75) (xy 163 60.5) (xy 157.75 77.75)
-				(xy 156.25 79) (xy 136.75 86) (xy 136.75 89) (xy 153 89) (xy 160.6 106.75) (xy 167.6 122.96) (xy 182 114.75)
+				(xy 128.75 93.5) (xy 126.75 93.5) (xy 126 93) (xy 126 91) (xy 127 90.5) (xy 127.25 81) (xy 133.75 79.75)
+				(xy 144.25 70.75) (xy 160.5 56.25) (xy 163.5 56.5) (xy 164.25 57) (xy 164.25 59.75) (xy 163 60.5)
+				(xy 157.75 77.75) (xy 156.25 79) (xy 135.5 85.91) (xy 135.5 89.09) (xy 153 89) (xy 160.6 106.75)
+				(xy 167.6 122.96) (xy 182 114.75)
 			)
 		)
