File: dc-to-dc-maker/dc-to-dc-boost-converter/dc-to-dc-buck-converter.kicad_sch (KiCad schematic)
At the start: 30 parts, among them IC1 LA_55-P, IC2 LA_55-P, IC3 EL7104CNZ, J2 Jgen, J3 Jaux 9V, J4 Jind, J5 Jout +50V, U1 IRF640NPBF

Commit message: update
Other:
- moved on the sheet: J4, J5
Changed lines of the file:
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@@
 	)
 	(junction
+		(at 194.31 50.8)
+		(diameter 0)
+		(color 0 0 0 0)
+	)
+	(junction
 		(at 269.24 115.57)
 		(diameter 0)
@@
 	)
 	(junction
-		(at 194.31 49.53)
-		(diameter 0)
-		(color 0 0 0 0)
-	)
-	(junction
 		(at 77.47 55.88)
 		(diameter 0)
@@
 	(wire
 		(pts
-			(xy 58.42 110.49) (xy 179.07 110.49)
+			(xy 58.42 110.49) (xy 177.8 110.49)
 		)
 		(stroke
@@
 	(wire
 		(pts
+			(xy 194.31 50.8) (xy 194.31 49.53)
+		)
+		(stroke
+			(width 0)
+			(type default)
+		)
+	)
+	(wire
+		(pts
 			(xy 138.43 50.8) (xy 138.43 58.42)
 		)
@@
 	(wire
 		(pts
+			(xy 191.77 50.8) (xy 191.77 64.77)
+		)
+		(stroke
+			(width 0)
+			(type default)
+		)
+	)
+	(wire
+		(pts
 			(xy 99.06 160.02) (xy 113.03 160.02)
 		)
@@
 	(wire
 		(pts
-			(xy 179.07 50.8) (xy 179.07 110.49)
+			(xy 177.8 50.8) (xy 177.8 110.49)
 		)
 		(stroke
@@
 	(wire
 		(pts
-			(xy 191.77 45.72) (xy 191.77 53.34)
-		)
-		(stroke
-			(width 0)
-			(type default)
-		)
-	)
-	(wire
-		(pts
 			(xy 113.03 160.02) (xy 113.03 175.26)
 		)
@@
 	(wire
 		(pts
-			(xy 181.61 68.58) (xy 204.47 68.58)
+			(xy 180.34 68.58) (xy 204.47 68.58)
 		)
 		(stroke
@@
 	(wire
 		(pts
-			(xy 194.31 45.72) (xy 194.31 49.53)
-		)
-		(stroke
-			(width 0)
-			(type default)
-		)
-	)
-	(wire
-		(pts
 			(xy 148.59 81.28) (xy 158.75 81.28)
 		)
@@
 	(wire
 		(pts
-			(xy 181.61 50.8) (xy 181.61 68.58)
+			(xy 180.34 50.8) (xy 180.34 68.58)
 		)
 		(stroke
@@
 	(wire
 		(pts
-			(xy 194.31 60.96) (xy 194.31 49.53)
+			(xy 194.31 60.96) (xy 194.31 50.8)
 		)
 		(stroke
@@
 	(symbol
 		(lib_id "1715721(screw connector):1715721")
-		(at 194.31 45.72 270)
+		(at 194.31 50.8 270)
 		(mirror x)
 		(unit 1)
@@
 		(dnp no)
 		(property "Reference" "J5"
-			(at 193.04 26.67 90)
+			(at 193.04 31.75 90)
 			(effects
 				(font
@@
 		)
 		(property "Value" "Jout +50V"
-			(at 193.04 28.448 90)
+			(at 193.04 33.528 90)
 			(effects
 				(font
@@
 		)
 		(property "Footprint" "1715721(screw connector):1715721"
-			(at 99.39 29.21 0)
+			(at 99.39 34.29 0)
 			(effects
 				(font
@@
 		)
 		(property "Datasheet" "http://www.phoenixcontact.com/de/produkte/1715721/pdf"
-			(at -0.61 29.21 0)
+			(at -0.61 34.29 0)
 			(effects
 				(font
@@
 		)
 		(property "Description" "PCB terminal block, nominal current: 17.5 A, rated voltage (III/2): 400 V, nominal cross section: 1.5 mm?, Number of potentials: 2, Number of rows: 1, Number of positions per row: 2, product range: MKDS 1,5, pitch: 5.08 mm, connection method: Screw connection with tension sleeve, mounting: Wave soldering, conductor/PCB connection direction: 0 ?, color: green, Pin layout: Linear pinning, Solder pin [P]: 3.5 mm, type of packaging: packed in cardboard. The article can be aligned to create different nos. of pos"
-			(at 194.31 45.72 0)
+			(at 194.31 50.8 0)
 			(effects
 				(font
@@
 		)
 		(property "Height" "13.95"
-			(at -200.61 29.21 0)
+			(at -200.61 34.29 0)
 			(effects
 				(font
@@
 		)
 		(property "Farnell Part Number" ""
-			(at -300.61 29.21 0)
+			(at -300.61 34.29 0)
 			(effects
 				(font
@@
 		)
 		(property "Farnell Price/Stock" ""
-			(at -400.61 29.21 0)
+			(at -400.61 34.29 0)
 			(effects
 				(font
@@
 		)
 		(property "Manufacturer_Name" "Phoenix Contact"
-			(at -500.61 29.21 0)
+			(at -500.61 34.29 0)
 			(effects
 				(font
@@
 		)
 		(property "Manufacturer_Part_Number" "1715721"
-			(at -600.61 29.21 0)
+			(at -600.61 34.29 0)
 			(effects
 				(font
@@
 	(symbol
 		(lib_id "power:GND")
-		(at 191.77 53.34 0)
+		(at 191.77 64.77 0)
 		(unit 1)
 		(exclude_from_sim no)
@@
 		(on_board yes)
 		(dnp no)
-		(fields_autoplaced yes)
 		(property "Reference" "#PWR011"
-			(at 191.77 59.69 0)
+			(at 191.77 71.12 0)
 			(effects
 				(font
@@
 		)
 		(property "Value" "GND"
-			(at 191.77 58.42 0)
+			(at 195.834 66.548 0)
 			(effects
 				(font
@@
 		)
 		(property "Footprint" ""
-			(at 191.77 53.34 0)
+			(at 191.77 64.77 0)
 			(effects
 				(font
@@
 		)
 		(property "Datasheet" ""
-			(at 191.77 53.34 0)
+			(at 191.77 64.77 0)
 			(effects
 				(font
@@
 		)
 		(property "Description" "Power symbol creates a global label with name \"GND\" , ground"
-			(at 191.77 53.34 0)
+			(at 191.77 64.77 0)
 			(effects
 				(font
@@
 	(symbol
 		(lib_id "1715721(screw connector):1715721")
-		(at 179.07 50.8 90)
+		(at 177.8 50.8 90)
 		(unit 1)
 		(exclude_from_sim no)
@@
 		(dnp no)
 		(property "Reference" "J4"
-			(at 180.34 31.75 90)
+			(at 179.07 31.75 90)
 			(effects
 				(font
@@
 		)
 		(property "Value" "Jind"
-			(at 180.34 33.528 90)
+			(at 179.07 33.528 90)
 			(effects
 				(font
@@
 		)
 		(property "Footprint" "1715721(screw connector):1715721"
-			(at 273.99 34.29 0)
+			(at 272.72 34.29 0)
 			(effects
 				(font
@@
 		)
 		(property "Datasheet" "http://www.phoenixcontact.com/de/produkte/1715721/pdf"
-			(at 373.99 34.29 0)
+			(at 372.72 34.29 0)
 			(effects
 				(font
@@
 		)
 		(property "Description" "PCB terminal block, nominal current: 17.5 A, rated voltage (III/2): 400 V, nominal cross section: 1.5 mm?, Number of potentials: 2, Number of rows: 1, Number of positions per row: 2, product range: MKDS 1,5, pitch: 5.08 mm, connection method: Screw connection with tension sleeve, mounting: Wave soldering, conductor/PCB connection direction: 0 ?, color: green, Pin layout: Linear pinning, Solder pin [P]: 3.5 mm, type of packaging: packed in cardboard. The article can be aligned to create different nos. of pos"
-			(at 179.07 50.8 0)
+			(at 177.8 50.8 0)
 			(effects
 				(font
@@
 		)
 		(property "Height" "13.95"
-			(at 573.99 34.29 0)
+			(at 572.72 34.29 0)
 			(effects
 				(font
@@
 		)
 		(property "Farnell Part Number" ""
-			(at 673.99 34.29 0)
+			(at 672.72 34.29 0)
 			(effects
 				(font
@@
 		)
 		(property "Farnell Price/Stock" ""
-			(at 773.99 34.29 0)
+			(at 772.72 34.29 0)
 			(effects
 				(font
@@
 		)
 		(property "Manufacturer_Name" "Phoenix Contact"
-			(at 873.99 34.29 0)
+			(at 872.72 34.29 0)
 			(effects
 				(font
@@
 		)
 		(property "Manufacturer_Part_Number" "1715721"
-			(at 973.99 34.29 0)
+			(at 972.72 34.29 0)
 			(effects
 				(font
